File: _saved_HolyIoT-NRF52840-Breakout.sch (KiCad schematic (older format))
At the start: 6 parts, among them J1 Conn_01x13_Male, J2 Conn_01x09_Male, J3 Conn_01x11_Male, J4 Conn_01x13_Male, J5 Conn_01x09_Male, U1 HolyIOT_NRF52840

Commit message: First Routing
First use if PCBNew on this board
Changed lines of the file:
@@
 $EndComp
 $Comp
-L power:GND #PWR?
+L power:GND #PWR0101
 U 1 1 5B8D035A
 P 4500 1750
-F 0 "#PWR?" H 4500 1500 50  0001 C CNN
+F 0 "#PWR0101" H 4500 1500 50  0001 C CNN
 F 1 "GND" H 4505 1577 50  0000 C CNN
 F 2 "" H 4500 1750 50  0001 C CNN
@@
 $EndComp
 $Comp
-L power:GND #PWR?
+L power:GND #PWR0102
 U 1 1 5B8D03CB
 P 7100 1800
-F 0 "#PWR?" H 7100 1550 50  0001 C CNN
+F 0 "#PWR0102" H 7100 1550 50  0001 C CNN
 F 1 "GND" H 7105 1627 50  0000 C CNN
 F 2 "" H 7100 1800 50  0001 C CNN
@@
 $EndComp
 $Comp
-L power:GND #PWR?
+L power:GND #PWR0103
 U 1 1 5B8D0406
 P 7850 3350
-F 0 "#PWR?" H 7850 3100 50  0001 C CNN
+F 0 "#PWR0103" H 7850 3100 50  0001 C CNN
 F 1 "GND" H 7855 3177 50  0000 C CNN
 F 2 "" H 7850 3350 50  0001 C CNN
@@
 	7850 3300 7850 3350
 Connection ~ 7300 3300
+$Comp
+L Serigraphie:LOGO #G1
+U 1 1 5B8EAD1C
+P 8350 5000
+F 0 "#G1" H 8350 4770 60  0001 C CNN
+F 1 "LOGO" H 8350 5230 60  0001 C CNN
+F 2 "MWL:Serigraphie" H 8350 5000 50  0001 C CNN
+F 3 "" H 8350 5000 50  0001 C CNN
+	1    8350 5000
+	1    0    0    -1
+$EndComp
 $EndSCHEMATC
