File: HolyIoT-NRF52840-Breakout.sch (KiCad schematic (older format))
At the start: 1 part

Commit message: Moving On
add datasheet + finished schematics
Parts:
- removed U?: HolyIOT_NRF52840, symbol MWL:HolyIOT_NRF52840
- added J1, J4: Conn_01x13_Male, Connector_PinSocket_2.54mm:PinSocket_1x13_P2.54mm_Vertical, symbol Connector:Conn_01x13_Male
- added J2, J5: Conn_01x09_Male, Connector_PinSocket_2.54mm:PinSocket_1x09_P2.54mm_Vertical, symbol Connector:Conn_01x09_Male
- added J3: Conn_01x11_Male, Connector_PinSocket_2.54mm:PinSocket_1x11_P2.54mm_Vertical, symbol Connector:Conn_01x11_Male
- added U1: HolyIOT_NRF52840, symbol MWL:HolyIOT_NRF52840
Connections:
- wire segments 0 -> 158

Commit message: First Routing
First use if PCBNew on this board
Parts:
- U1: footprint (none) -> MWL:HolyIOT-NRF52840-Module
Connections:
- net labels added: GND
- wire segments 158 -> 168
Changed lines of the file:
@@
 	6650 2700 6650 2050
 Wire Wire Line
-	6650 2050 7400 2050
+	6650 2050 6800 2050
 Wire Wire Line
 	4950 3750 4850 3750
@@
 	4850 2700 4850 2050
 Wire Wire Line
-	4850 2050 4150 2050
+	4850 2050 4700 2050
 $Comp
 L MWL:HolyIOT_NRF52840 U1
@@
 F 0 "U1" H 5750 4265 50  0000 C CNN
 F 1 "HolyIOT_NRF52840" H 5750 4174 50  0000 C CNN
-F 2 "" H 5750 3250 50  0001 C CNN
+F 2 "MWL:HolyIOT-NRF52840-Module" H 5750 3250 50  0001 C CNN
 F 3 "" H 5750 3250 50  0001 C CNN
 	1    5750 3250
 	1    0    0    -1
 $EndComp
+$Comp
+L power:GND #PWR0101
+U 1 1 5B8D035A
+P 4500 1750
+F 0 "#PWR0101" H 4500 1500 50  0001 C CNN
+F 1 "GND" H 4505 1577 50  0000 C CNN
+F 2 "" H 4500 1750 50  0001 C CNN
+F 3 "" H 4500 1750 50  0001 C CNN
+	1    4500 1750
+	1    0    0    -1
+$EndComp
+$Comp
+L power:GND #PWR0102
+U 1 1 5B8D03CB
+P 7100 1800
+F 0 "#PWR0102" H 7100 1550 50  0001 C CNN
+F 1 "GND" H 7105 1627 50  0000 C CNN
+F 2 "" H 7100 1800 50  0001 C CNN
+F 3 "" H 7100 1800 50  0001 C CNN
+	1    7100 1800
+	1    0    0    -1
+$EndComp
+$Comp
+L power:GND #PWR0103
+U 1 1 5B8D0406
+P 7850 3350
+F 0 "#PWR0103" H 7850 3100 50  0001 C CNN
+F 1 "GND" H 7855 3177 50  0000 C CNN
+F 2 "" H 7850 3350 50  0001 C CNN
+F 3 "" H 7850 3350 50  0001 C CNN
+	1    7850 3350
+	1    0    0    -1
+$EndComp
+Wire Wire Line
+	4700 2050 4700 1650
+Wire Wire Line
+	4700 1650 4500 1650
+Wire Wire Line
+	4500 1650 4500 1750
+Connection ~ 4700 2050
+Wire Wire Line
+	4700 2050 4150 2050
+Wire Wire Line
+	6800 2050 6800 1700
+Wire Wire Line
+	6800 1700 7100 1700
+Wire Wire Line
+	7100 1700 7100 1800
+Connection ~ 6800 2050
+Wire Wire Line
+	6800 2050 7400 2050
+Wire Wire Line
+	7300 3300 7850 3300
+Wire Wire Line
+	7850 3300 7850 3350
+Connection ~ 7300 3300
+$Comp
+L Serigraphie:LOGO #G?
+U 1 1 5B8EAD1C
+P 8350 5000
+F 0 "#G?" H 8350 4770 60  0001 C CNN
+F 1 "LOGO" H 8350 5230 60  0001 C CNN
+F 2 "MWL:Serigraphie" H 8350 5000 50  0001 C CNN
+F 3 "" H 8350 5000 50  0001 C CNN
+	1    8350 5000
+	1    0    0    -1
+$EndComp

Commit message: Routing done
Last thing to do : labelling
Parts:
- removed J1, J4: Conn_01x13_Male, Connector_PinSocket_2.54mm:PinSocket_1x13_P2.54mm_Vertical, symbol Connector:Conn_01x13_Male
- removed J2, J5: Conn_01x09_Male, Connector_PinSocket_2.54mm:PinSocket_1x09_P2.54mm_Vertical, symbol Connector:Conn_01x09_Male
- added J1, J2: Conn_01x22_Male, Connector_PinHeader_2.54mm:PinHeader_1x22_P2.54mm_Vertical, symbol Connector:Conn_01x22_Male
Changed lines of the file:
@@
 $EndDescr
-$Comp
-L Connector:Conn_01x13_Male J1
-U 1 1 5B8BEF03
-P 3950 2650
-F 0 "J1" H 3350 2800 50  0000 C CNN
-F 1 "Conn_01x13_Male" H 3350 2650 50  0000 C CNN
-F 2 "Connector_PinSocket_2.54mm:PinSocket_1x13_P2.54mm_Vertical" H 3950 2650 50  0001 C CNN
-F 3 "~" H 3950 2650 50  0001 C CNN
-	1    3950 2650
-	1    0    0    -1
-$EndComp
-$Comp
-L Connector:Conn_01x13_Male J4
-U 1 1 5B8BEFAD
-P 7600 2650
-F 0 "J4" H 7573 2673 50  0000 R CNN
-F 1 "Conn_01x13_Male" H 7573 2582 50  0000 R CNN
-F 2 "Connector_PinSocket_2.54mm:PinSocket_1x13_P2.54mm_Vertical" H 7600 2650 50  0001 C CNN
-F 3 "~" H 7600 2650 50  0001 C CNN
-	1    7600 2650
-	-1   0    0    -1
-$EndComp
-$Comp
-L Connector:Conn_01x09_Male J2
-U 1 1 5B8BF0D5
-P 3950 3750
-F 0 "J2" H 3500 3900 50  0000 C CNN
-F 1 "Conn_01x09_Male" H 3500 3750 50  0000 C CNN
-F 2 "Connector_PinSocket_2.54mm:PinSocket_1x09_P2.54mm_Vertical" H 3950 3750 50  0001 C CNN
-F 3 "~" H 3950 3750 50  0001 C CNN
-	1    3950 3750
-	1    0    0    -1
-$EndComp
-$Comp
-L Connector:Conn_01x09_Male J5
-U 1 1 5B8BF16B
-P 7600 3750
-F 0 "J5" H 7573 3773 50  0000 R CNN
-F 1 "Conn_01x09_Male" H 7573 3682 50  0000 R CNN
-F 2 "Connector_PinSocket_2.54mm:PinSocket_1x09_P2.54mm_Vertical" H 7600 3750 50  0001 C CNN
-F 3 "~" H 7600 3750 50  0001 C CNN
-	1    7600 3750
-	-1   0    0    -1
-$EndComp
 $Comp
 L Connector:Conn_01x11_Male J3
@@
 Connection ~ 7300 3300
 $Comp
-L Serigraphie:LOGO #G?
-U 1 1 5B8EAD1C
-P 8350 5000
-F 0 "#G?" H 8350 4770 60  0001 C CNN
-F 1 "LOGO" H 8350 5230 60  0001 C CNN
-F 2 "MWL:Serigraphie" H 8350 5000 50  0001 C CNN
-F 3 "" H 8350 5000 50  0001 C CNN
-	1    8350 5000
+L Connector:Conn_01x22_Male J1
+U 1 1 5B8F408A
+P 3950 3050
+F 0 "J1" H 3450 3700 50  0000 C CNN
+F 1 "Conn_01x22_Male" H 3450 3450 50  0000 C CNN
+F 2 "Connector_PinHeader_2.54mm:PinHeader_1x22_P2.54mm_Vertical" H 3950 3050 50  0001 C CNN
+F 3 "~" H 3950 3050 50  0001 C CNN
+	1    3950 3050
 	1    0    0    -1
 $EndComp
+$Comp
+L Connector:Conn_01x22_Male J2
+U 1 1 5B90F2A0
+P 7600 3050
+F 0 "J2" H 7150 2750 50  0000 C CNN
+F 1 "Conn_01x22_Male" H 7100 2950 50  0000 C CNN
+F 2 "Connector_PinHeader_2.54mm:PinHeader_1x22_P2.54mm_Vertical" H 7600 3050 50  0001 C CNN
+F 3 "~" H 7600 3050 50  0001 C CNN
+	1    7600 3050
+	-1   0    0    -1
+$EndComp
 $EndSCHEMATC

Commit message: micro-usb b
add micro-usb
Parts:
- added C1: C, MWL:SM0805, symbol Device:C_Small
- added P1: USB_micro_B, MWL:USB_Micro-B, symbol MWL:USB_micro_B
- added R1, R2: R, MWL:SM0805, symbol Device:R
Connections:
- wire segments 168 -> 192
- no-connect marks 0 -> 1
Changed lines of the file:
@@
 L Connector:Conn_01x11_Male J3
 U 1 1 5B8BF522
-P 5700 4600
-F 0 "J3" V 5628 4577 50  0000 C CNN
-F 1 "Conn_01x11_Male" V 5537 4577 50  0000 C CNN
-F 2 "Connector_PinSocket_2.54mm:PinSocket_1x11_P2.54mm_Vertical" H 5700 4600 50  0001 C CNN
-F 3 "~" H 5700 4600 50  0001 C CNN
-	1    5700 4600
+P 5700 5950
+F 0 "J3" V 5650 6550 50  0000 C CNN
+F 1 "Conn_01x11_Male" V 5550 6550 50  0000 C CNN
+F 2 "Connector_PinSocket_2.54mm:PinSocket_1x11_P2.54mm_Vertical" H 5700 5950 50  0001 C CNN
+F 3 "~" H 5700 5950 50  0001 C CNN
+	1    5700 5950
 	0    -1   -1   0
 $EndComp
@@
 	5500 4050 5200 4050
 Wire Wire Line
-	5200 4050 5200 4400
-Wire Wire Line
 	5550 4000 5550 4100
 Wire Wire Line
 	5550 4100 5300 4100
 Wire Wire Line
-	5300 4100 5300 4400
-Wire Wire Line
-	6000 4000 6200 4000
-Wire Wire Line
-	6200 4000 6200 4400
+	6000 4000 6500 4000
 Wire Wire Line
 	5950 4000 5950 4050
 Wire Wire Line
-	5950 4050 6100 4050
-Wire Wire Line
-	6100 4050 6100 4400
+	5950 4050 6300 4050
 Wire Wire Line
 	5900 4000 5900 4100
@@
 	5900 4100 6000 4100
 Wire Wire Line
-	6000 4100 6000 4400
-Wire Wire Line
 	5850 4000 5850 4150
 Wire Wire Line
 	5850 4150 5900 4150
 Wire Wire Line
-	5900 4150 5900 4400
-Wire Wire Line
-	5800 4000 5800 4400
-Wire Wire Line
-	5400 4400 5400 4150
-Wire Wire Line
 	5400 4150 5600 4150
 Wire Wire Line
 	5600 4150 5600 4000
 Wire Wire Line
-	5500 4400 5500 4200
-Wire Wire Line
 	5500 4200 5650 4200
 Wire Wire Line
@@
 	5700 4250 5600 4250
 Wire Wire Line
-	5600 4250 5600 4400
-Wire Wire Line
 	5700 4000 5700 4250
 Wire Wire Line
 	5750 4350 5700 4350
-Wire Wire Line
-	5700 4350 5700 4400
 Wire Wire Line
 	5750 4000 5750 4350
@@
 	-1   0    0    -1
 $EndComp
+$Comp
+L MWL:USB_micro_B P1
+U 1 1 5B9479BF
+P 7350 5050
+F 0 "P1" H 7500 5050 60  0000 L CNN
+F 1 "USB_micro_B" H 7500 5200 60  0000 L CNN
+F 2 "MWL:USB_Micro-B" H 7350 5050 60  0001 C CNN
+F 3 "" H 7350 5050 60  0000 C CNN
+	1    7350 5050
+	1    0    0    -1
+$EndComp
+$Comp
+L Device:R R1
+U 1 1 5B963139
+P 6300 4550
+F 0 "R1" H 6250 4700 50  0000 L CNN
+F 1 "R" H 6200 4550 50  0000 L CNN
+F 2 "MWL:SM0805" V 6230 4550 50  0001 C CNN
+F 3 "~" H 6300 4550 50  0001 C CNN
+	1    6300 4550
+	1    0    0    -1
+$EndComp
+$Comp
+L Device:R R2
+U 1 1 5B963171
+P 6500 4550
+F 0 "R2" H 6450 4700 50  0000 L CNN
+F 1 "R" H 6550 4550 50  0000 L CNN
+F 2 "MWL:SM0805" V 6430 4550 50  0001 C CNN
+F 3 "~" H 6500 4550 50  0001 C CNN
+	1    6500 4550
+	1    0    0    -1
+$EndComp
+Wire Wire Line
+	7000 4850 6800 4850
+Wire Wire Line
+	6800 4850 6800 4450
+$Comp
+L power:GND #PWR01
+U 1 1 5B97F26D
+P 6950 4450
+F 0 "#PWR01" H 6950 4200 50  0001 C CNN
+F 1 "GND" H 6955 4277 50  0000 C CNN
+F 2 "" H 6950 4450 50  0001 C CNN
+F 3 "" H 6950 4450 50  0001 C CNN
+	1    6950 4450
+	0    -1   -1   0
+$EndComp
+NoConn ~ 7000 4950
+$Comp
+L Device:C_Small C1
+U 1 1 5BA02818
+P 6100 4800
+F 0 "C1" H 5850 4850 50  0000 L CNN
+F 1 "C" H 5900 4750 50  0000 L CNN
+F 2 "MWL:SM0805" H 6138 4650 50  0001 C CNN
+F 3 "~" H 6100 4800 50  0001 C CNN
+	1    6100 4800
+	0    -1   -1   0
+$EndComp
+Wire Wire Line
+	6300 4050 6300 4400
+Wire Wire Line
+	6500 4000 6500 4400
+Wire Wire Line
+	5200 4050 5200 5750
+Wire Wire Line
+	5300 4100 5300 5750
+Wire Wire Line
+	5400 4150 5400 5750
+Wire Wire Line
+	5500 4200 5500 5750
+Wire Wire Line
+	5600 4250 5600 5750
+Wire Wire Line
+	5700 4350 5700 5750
+Wire Wire Line
+	5800 4000 5800 5750
+Wire Wire Line
+	5900 4150 5900 5750
+Wire Wire Line
+	6800 4450 6950 4450
+Wire Wire Line
+	6500 5050 7000 5050
+Wire Wire Line
+	6500 5600 6200 5600
+Wire Wire Line
+	6200 5600 6200 5750
+Wire Wire Line
+	6300 5150 7000 5150
+Wire Wire Line
+	6300 5500 6100 5500
+Wire Wire Line
+	6100 5500 6100 5750
+Wire Wire Line
+	6300 4700 6300 5150
+Wire Wire Line
+	6500 4700 6500 5050
+Connection ~ 6500 5050
+Wire Wire Line
+	6500 5050 6500 5600
+Connection ~ 6300 5150
+Wire Wire Line
+	6300 5150 6300 5500
+Wire Wire Line
+	6200 4800 6250 4800
+$Comp
+L power:GND #PWR02
+U 1 1 5BBFC2FE
+P 6100 4600
+F 0 "#PWR02" H 6100 4350 50  0001 C CNN
+F 1 "GND" H 6105 4427 50  0000 C CNN
+F 2 "" H 6100 4600 50  0001 C CNN
+F 3 "" H 6100 4600 50  0001 C CNN
+	1    6100 4600
+	-1   0    0    1
+$EndComp
+Wire Wire Line
+	6000 5750 6000 5450
+Wire Wire Line
+	6000 5450 5950 5450
+Wire Wire Line
+	5950 5450 5950 5250
+Wire Wire Line
+	5950 4900 6000 4900
+Wire Wire Line
+	6000 4900 6000 4800
+Wire Wire Line
+	6000 4100 6000 4800
+Connection ~ 6000 4800
+Wire Wire Line
+	6250 4800 6250 4700
+Wire Wire Line
+	6250 4700 6100 4700
+Wire Wire Line
+	6100 4700 6100 4600
+Wire Wire Line
+	5950 5250 7000 5250
+Connection ~ 5950 5250
+Wire Wire Line
+	5950 5250 5950 4900
 $EndSCHEMATC

Commit message: Morning Routing is always the best...
 - Routing DONE in 2 Layers
- Verification has to be done before order...
Parts:
- removed J2: Conn_01x22_Male, Connector_PinHeader_2.54mm:PinHeader_1x22_P2.54mm_Vertical, symbol Connector:Conn_01x22_Male
- removed J3: Conn_01x11_Male, Connector_PinSocket_2.54mm:PinSocket_1x11_P2.54mm_Vertical, symbol Connector:Conn_01x11_Male
- added C2: C, MWL:SM0805, symbol Device:C_Small
- added J2: Conn_01x18_Male, Connector_PinHeader_2.54mm:PinHeader_1x18_P2.54mm_Vertical, symbol Connector:Conn_01x18_Male
- added J3: Conn_01x07_Male, Connector_PinHeader_2.54mm:PinHeader_1x07_P2.54mm_Vertical, symbol Connector:Conn_01x07_Male
- added J4: Prog, Connector_PinHeader_1.27mm:PinHeader_2x05_P1.27mm_Vertical_SMD, symbol Connector_Generic_MountingPin:Conn_02x05_Odd_Even_MountingPin
Connections:
- net labels added: SWDCLK, SWDIO, V_NRF
- wire segments 192 -> 211
- no-connect marks 1 -> 8
Other:
- note added: "Program"

Commit message: Generate Gerber
Generate Gerber
Rework Edge.Cut
Parts:
- added G1: LOGO, MWL:Serigraphie, symbol Serigraphie:LOGO
Changed lines of the file:
@@
 Wire Wire Line
 	4850 4650 4850 4800
+$Comp
+L Serigraphie:LOGO G1
+U 1 1 5B9AE5DB
+P 1750 4700
+F 0 "G1" H 1750 4470 60  0001 C CNN
+F 1 "LOGO" H 1750 4930 60  0001 C CNN
+F 2 "MWL:Serigraphie" H 1750 4700 50  0001 C CNN
+F 3 "" H 1750 4700 50  0001 C CNN
+	1    1750 4700
+	1    0    0    -1
+$EndComp
 $EndSCHEMATC

Commit message: Change after Rev 1.0
Need some check for 1.1

Do we had some sensors???
Parts:
- removed C1: C, MWL:SM0805, symbol Device:C_Small
- removed P1: USB_micro_B, MWL:USB_Micro-B, symbol MWL:USB_micro_B
- removed R1, R2: R, MWL:SM0805, symbol Device:R
- added J5: Prog, Connector_PinHeader_2.54mm:PinHeader_1x06_P2.54mm_Vertical, symbol Connector:Conn_01x06_Male
- J3: value Conn_01x07_Male -> Conn_01x10_Male; footprint Connector_PinHeader_2.54mm:PinHeader_1x07_P2.54mm_Vertical -> Connector_PinHeader_2.54mm:PinHeader_1x10_P2.54mm_Vertical; symbol Connector:Conn_01x07_Male -> Connector:Conn_01x10_Male
Connections:
- wire segments 211 -> 212
- no-connect marks 8 -> 7
Other:
- note added: "Program 2.54mm Format"
- note added: "Program CMS Format"
- note removed: "Program"
Changed lines of the file:
@@
 	5550 4100 5300 4100
 Wire Wire Line
-	6000 4000 6500 4000
-Wire Wire Line
-	5950 4000 5950 4050
-Wire Wire Line
-	5950 4050 6300 4050
-Wire Wire Line
-	5900 4000 5900 4100
-Wire Wire Line
-	5900 4100 6000 4100
-Wire Wire Line
-	5850 4000 5850 4150
-Wire Wire Line
-	5850 4150 5900 4150
+	5850 4000 5850 4300
+Wire Wire Line
+	5850 4300 5900 4300
 Wire Wire Line
 	5400 4150 5600 4150
@@
 	1    0    0    -1
 $EndComp
-$Comp
-L MWL:USB_micro_B P1
-U 1 1 5B9479BF
-P 6250 6200
-F 0 "P1" H 6400 6200 60  0000 L CNN
-F 1 "USB_micro_B" H 6400 6350 60  0000 L CNN
-F 2 "MWL:USB_Micro-B" H 6250 6200 60  0001 C CNN
-F 3 "" H 6250 6200 60  0000 C CNN
-	1    6250 6200
-	0    1    1    0
-$EndComp
-$Comp
-L Device:R R1
-U 1 1 5B963139
-P 6300 4550
-F 0 "R1" H 6250 4700 50  0000 L CNN
-F 1 "R" H 6200 4550 50  0000 L CNN
-F 2 "MWL:SM0805" V 6230 4550 50  0001 C CNN
-F 3 "~" H 6300 4550 50  0001 C CNN
-	1    6300 4550
-	1    0    0    -1
-$EndComp
-$Comp
-L Device:R R2
-U 1 1 5B963171
-P 6500 4550
-F 0 "R2" H 6450 4700 50  0000 L CNN
-F 1 "R" H 6550 4550 50  0000 L CNN
-F 2 "MWL:SM0805" V 6430 4550 50  0001 C CNN
-F 3 "~" H 6500 4550 50  0001 C CNN
-	1    6500 4550
-	1    0    0    -1
-$EndComp
-Wire Wire Line
-	6450 5850 6450 5650
-Wire Wire Line
-	6450 5650 6850 5650
-$Comp
-L power:GND #PWR01
-U 1 1 5B97F26D
-P 6850 5800
-F 0 "#PWR01" H 6850 5550 50  0001 C CNN
-F 1 "GND" H 6855 5627 50  0000 C CNN
-F 2 "" H 6850 5800 50  0001 C CNN
-F 3 "" H 6850 5800 50  0001 C CNN
-	1    6850 5800
-	1    0    0    -1
-$EndComp
-NoConn ~ 6350 5850
-$Comp
-L Device:C_Small C1
-U 1 1 5BA02818
-P 6100 4550
-F 0 "C1" H 6100 4700 50  0000 L CNN
-F 1 "C" H 6150 4500 50  0000 L CNN
-F 2 "MWL:SM0805" H 6138 4400 50  0001 C CNN
-F 3 "~" H 6100 4550 50  0001 C CNN
-	1    6100 4550
-	1    0    0    -1
-$EndComp
-Wire Wire Line
-	6300 4050 6300 4400
-Wire Wire Line
-	6500 4000 6500 4400
 Wire Wire Line
 	5300 4100 5300 5750
@@
 	5800 4000 5800 5750
 Wire Wire Line
-	5900 4150 5900 5750
-Wire Wire Line
-	6850 5650 6850 5800
-Wire Wire Line
-	6300 4700 6300 5150
-$Comp
-L power:GND #PWR02
-U 1 1 5BBFC2FE
-P 6150 4900
-F 0 "#PWR02" H 6150 4650 50  0001 C CNN
-F 1 "GND" H 6155 4727 50  0000 C CNN
-F 2 "" H 6150 4900 50  0001 C CNN
-F 3 "" H 6150 4900 50  0001 C CNN
-	1    6150 4900
-	1    0    0    -1
-$EndComp
-Wire Wire Line
-	5950 4900 6000 4900
+	5900 4300 5900 5750
 $Comp
 L Connector_Generic_MountingPin:Conn_02x05_Odd_Even_MountingPin J4
@@
 NoConn ~ 2800 6750
 Text Notes 2400 5850 0    50   ~ 0
-Program
+Program CMS Format
 Text GLabel 7750 2550 2    50   Input ~ 0
 SWDIO
@@
 	6750 2150 8600 2150
 $Comp
-L Connector:Conn_01x07_Male J3
+L Connector:Conn_01x10_Male J3
 U 1 1 5BDB0FFD
-P 5600 5950
-F 0 "J3" V 5528 5927 50  0000 C CNN
-F 1 "Conn_01x07_Male" V 5400 6050 50  0000 C CNN
-F 2 "Connector_PinHeader_2.54mm:PinHeader_1x07_P2.54mm_Vertical" H 5600 5950 50  0001 C CNN
-F 3 "~" H 5600 5950 50  0001 C CNN
-	1    5600 5950
+P 5700 5950
+F 0 "J3" V 5628 5927 50  0000 C CNN
+F 1 "Conn_01x10_Male" V 5500 6050 50  0000 C CNN
+F 2 "Connector_PinHeader_2.54mm:PinHeader_1x10_P2.54mm_Vertical" H 5700 5950 50  0001 C CNN
+F 3 "~" H 5700 5950 50  0001 C CNN
+	1    5700 5950
 	0    -1   -1   0
 $EndComp
 Wire Wire Line
-	5950 5700 6050 5700
-Wire Wire Line
-	6050 5700 6050 5850
-Wire Wire Line
-	5950 4900 5950 5700
-Wire Wire Line
-	6150 5850 6150 5150
-Wire Wire Line
-	6150 5150 6300 5150
-Wire Wire Line
-	6250 5850 6250 5400
-Wire Wire Line
-	6250 5400 6500 5400
-Wire Wire Line
-	6500 4700 6500 5400
-Wire Wire Line
 	5200 4050 5200 4350
-Wire Wire Line
-	6000 4100 6000 4300
-Wire Wire Line
-	6100 4650 6100 4850
-Wire Wire Line
-	6100 4850 6150 4850
-Wire Wire Line
-	6150 4850 6150 4900
-Wire Wire Line
-	6100 4450 6100 4300
-Wire Wire Line
-	6100 4300 6000 4300
-Connection ~ 6000 4300
-Wire Wire Line
-	6000 4300 6000 4900
 Wire Wire Line
 	5200 4350 4850 4350
@@
 L Serigraphie:LOGO G1
 U 1 1 5B9AE5DB
-P 1750 4700
-F 0 "G1" H 1750 4470 60  0001 C CNN
-F 1 "LOGO" H 1750 4930 60  0001 C CNN
-F 2 "MWL:Serigraphie" H 1750 4700 50  0001 C CNN
-F 3 "" H 1750 4700 50  0001 C CNN
-	1    1750 4700
-	1    0    0    -1
-$EndComp
+P 5700 1500
+F 0 "G1" H 5700 1270 60  0001 C CNN
+F 1 "LOGO" H 5700 1730 60  0001 C CNN
+F 2 "MWL:Serigraphie" H 5700 1500 50  0001 C CNN
+F 3 "" H 5700 1500 50  0001 C CNN
+	1    5700 1500
+	1    0    0    -1
+$EndComp
+Wire Wire Line
+	5900 4000 5900 4200
+Wire Wire Line
+	5900 4200 6000 4200
+Wire Wire Line
+	6000 4200 6000 5750
+Wire Wire Line
+	5950 4000 5950 4150
+Wire Wire Line
+	5950 4150 6100 4150
+Wire Wire Line
+	6100 4150 6100 5750
+Wire Wire Line
+	6200 4050 6200 5750
+Wire Wire Line
+	6000 4000 6000 4050
+Wire Wire Line
+	6000 4050 6200 4050
+$Comp
+L Connector:Conn_01x06_Male J5
+U 1 1 5BDD1794
+P 2300 3800
+F 0 "J5" H 2350 4217 50  0000 C CNN
+F 1 "Prog" H 2350 4126 50  0000 C CNN
+F 2 "Connector_PinHeader_2.54mm:PinHeader_1x06_P2.54mm_Vertical" H 2300 3800 50  0001 C CNN
+F 3 "~" H 2300 3800 50  0001 C CNN
+	1    2300 3800
+	0    1    1    0
+$EndComp
+Text GLabel 1600 4200 0    50   Input ~ 0
+V_NRF
+$Comp
+L power:GND #PWR01
+U 1 1 5BDD179B
+P 1450 4450
+F 0 "#PWR01" H 1450 4200 50  0001 C CNN
+F 1 "GND" H 1455 4277 50  0000 C CNN
+F 2 "" H 1450 4450 50  0001 C CNN
+F 3 "" H 1450 4450 50  0001 C CNN
+	1    1450 4450
+	1    0    0    -1
+$EndComp
+Text GLabel 3000 4200 2    50   Input ~ 0
+SWDIO
+Text GLabel 3000 4400 2    50   Input ~ 0
+SWDCLK
+Wire Notes Line
+	600  3500 600  5300
+Wire Notes Line
+	600  5300 3750 5300
+Wire Notes Line
+	3750 5300 3750 3500
+Wire Notes Line
+	3750 3500 600  3500
+Wire Wire Line
+	1450 4300 1450 4450
+Wire Wire Line
+	2500 4200 3000 4200
+Wire Wire Line
+	2850 4300 2850 4400
+Wire Wire Line
+	2850 4400 3000 4400
+Text Notes 2100 3700 0    50   ~ 0
+Program 2.54mm Format
+Wire Wire Line
+	2100 4000 2100 4100
+Wire Wire Line
+	2100 4100 2050 4100
+Wire Wire Line
+	2050 4100 2050 4200
+Wire Wire Line
+	1600 4200 2050 4200
+Wire Wire Line
+	2000 4000 2000 4100
+Wire Wire Line
+	2000 4100 2050 4100
+Connection ~ 2050 4100
+Wire Wire Line
+	2250 4300 2250 4100
+Wire Wire Line
+	2250 4100 2200 4100
+Wire Wire Line
+	2200 4100 2200 4000
+Wire Wire Line
+	1450 4300 2250 4300
+Wire Wire Line
+	2300 4000 2300 4100
+Wire Wire Line
+	2300 4100 2250 4100
+Connection ~ 2250 4100
+Wire Wire Line
+	2500 4200 2500 4000
+Wire Wire Line
+	2400 4300 2400 4000
+Wire Wire Line
+	2400 4300 2850 4300
 $EndSCHEMATC
