File: HolyIoT-NRF52840-Breakout.kicad_pcb (KiCad board)
At the start: 2 copper layers, 45 x 60 mm, 12 parts, among them J1 Conn_01x22_Male, J2 Conn_01x18_Male, J3 Conn_01x07_Male, J4 Prog, P1 USB_micro_B, U1 HolyIOT_NRF52840

Commit message: Change after Rev 1.0
Need some check for 1.1

Do we had some sensors???
Parts:
- removed C1: C, MWL:SM0805
- removed P1: USB_micro_B, MWL:USB_Micro-B
- removed R1, R2: R, MWL:SM0805
- added J5: Prog, Connector_PinHeader_2.54mm:PinHeader_1x06_P2.54mm_Vertical, F.Cu at (123.4, 117.0)
- J3: value Conn_01x07_Male -> Conn_01x10_Male; footprint Connector_PinHeader_2.54mm:PinHeader_1x07_P2.54mm_Vertical -> Connector_PinHeader_2.54mm:PinHeader_1x10_P2.54mm_Vertical
- moved G1 17.8 mm to (131.6, 134.8) (x2)
- moved J4 15.2 mm to (126.4, 124.8)
- moved C2 1.45 mm to (109.6, 103.6)
Connections:
- J4 pad 10: (no net) -> Net-(J4-Pad10)
- J4 pad 5: (no net) -> Net-(J4-Pad5)
- J4 pad 6: (no net) -> Net-(J4-Pad6)
- J4 pad 7: (no net) -> Net-(J4-Pad7)
- J4 pad 8: (no net) -> Net-(J4-Pad8)
- J4 pad 9: (no net) -> Net-(J4-Pad9)
- U1 pad 45: Net-(R2-Pad1) -> Net-(J3-Pad10)
- U1 pad 46: Net-(R1-Pad1) -> Net-(J3-Pad9)
- U1 pad 47: Net-(C1-Pad1) -> Net-(J3-Pad8)
Routing:
- net Net-(C1-Pad1): track 56.0 -> 0.00 mm, vias 2 -> 0
- net Net-(J3-Pad10): track 0.00 -> 43.3 mm
- net Net-(J3-Pad9): track 0.00 -> 40.7 mm
- net Net-(R2-Pad1): track 38.5 -> 0.00 mm
- net Net-(J3-Pad8): track 0.00 -> 38.0 mm
- net Net-(R1-Pad1): track 37.5 -> 0.00 mm
- net SWDCLK: track 26.2 -> 47.3 mm
- net V_NRF: track 23.5 -> 43.9 mm
- net SWDIO: track 24.1 -> 43.7 mm, vias 2 -> 4
- net Net-(P1-Pad2): track 14.1 -> 0.00 mm
- net Net-(P1-Pad3): track 11.7 -> 0.00 mm
- net Net-(J2-Pad15): track 20.0 -> 15.9 mm
- net Net-(J2-Pad16): track 18.0 -> 15.4 mm
- net Net-(J2-Pad17): track 16.3 -> 14.7 mm
- net Net-(J2-Pad18): track 15.2 -> 14.2 mm
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Other:
- board text added: "D+"
- board text added: "D-"
- board text added: "SWDCLK"
- board text added: "SWDIO"
- board text added: "V1.1"
- board text added: "VBUS (5V)"
- board text added: "VDD (3V)"
- board text removed: "V1.0"

Commit message: Polish
Polish
Parts:
- added REF**: Bosch_LGA-8_2.5x2.5mm_P0.65mm_ClockwisePinNumbering, Package_LGA:Bosch_LGA-8_2.5x2.5mm_P0.65mm_ClockwisePinNumbering, F.Cu at (121.2, 134.0)
Changed lines of the file:
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@@
   (general
     (thickness 1.6)
-    (drawings 131)
+    (drawings 127)
     (tracks 396)
     (zones 0)
-    (modules 9)
+    (modules 10)
     (nets 60)
   )
@@
   (module MWL:Serigraphie (layer B.Cu)
     (at 131.6 134.8 180)
-    (fp_text reference G1 (at -4.6 -0.7 180) (layer B.SilkS) hide
+    (fp_text reference G1 (at -27.4 25.8 180) (layer B.SilkS) hide
       (effects (font (size 1.524 1.524) (thickness 0.3)) (justify mirror))
     )
-    (fp_text value LOGO (at 0.2 -1.3 180) (layer B.SilkS) hide
+    (fp_text value LOGO (at -27.2 22.8 180) (layer B.SilkS) hide
       (effects (font (size 1.524 1.524) (thickness 0.3)) (justify mirror))
     )
@@
       (effects (font (size 1 1) (thickness 0.15)))
     )
-    (fp_text value Conn_01x22_Male (at 61.4 12.6) (layer F.Fab)
+    (fp_text value Conn_01x22_Male (at 60.6 12.6) (layer F.Fab)
       (effects (font (size 1 1) (thickness 0.15)))
     )
@@
   (module MWL:Serigraphie (layer F.Cu)
     (at 131.6 134.8)
-    (fp_text reference G1 (at 0 0) (layer F.SilkS) hide
+    (fp_text reference G1 (at 27.4 -19.8) (layer F.SilkS) hide
       (effects (font (size 1.524 1.524) (thickness 0.3)))
     )
-    (fp_text value LOGO (at 0.75 0) (layer F.SilkS) hide
+    (fp_text value LOGO (at 27.2 -17.2) (layer F.SilkS) hide
       (effects (font (size 1.524 1.524) (thickness 0.3)))
     )
@@
     )
   )
-  (gr_text SWDIO (at 131.4 122.2) (layer B.SilkS)
-    (effects (font (size 0.5 0.5) (thickness 0.1)) (justify mirror))
-  )
-  (gr_text SWDCLK (at 131.8 123.4) (layer B.SilkS)
-    (effects (font (size 0.5 0.5) (thickness 0.1)) (justify mirror))
-  )
-  (gr_text GND (at 121.6 123.6) (layer B.SilkS)
-    (effects (font (size 0.5 0.5) (thickness 0.1)) (justify mirror))
-  )
-  (gr_text "VDD (3V)" (at 120.8 122.2) (layer B.SilkS)
-    (effects (font (size 0.5 0.5) (thickness 0.1)) (justify mirror))
+  (module Package_LGA:Bosch_LGA-8_2.5x2.5mm_P0.65mm_ClockwisePinNumbering (layer F.Cu)
+    (at 121.2 134 270)
+    (descr LGA-8)
+    (tags "lga land grid array")
+    (attr smd)
+    (fp_text reference REF** (at 0.015 -2.465 270) (layer F.SilkS)
+      (effects (font (size 1 1) (thickness 0.15)))
+    )
+    (fp_text value Bosch_LGA-8_2.5x2.5mm_P0.65mm_ClockwisePinNumbering (at 0.015 2.535 270) (layer F.Fab)
+      (effects (font (size 1 1) (thickness 0.15)))
+    )
+    (fp_line (start 1.41 1.54) (end -1.41 1.54) (layer F.CrtYd) (width 0.05))
+    (fp_line (start 1.41 -1.54) (end 1.41 1.54) (layer F.CrtYd) (width 0.05))
+    (fp_line (start -1.41 -1.54) (end 1.41 -1.54) (layer F.CrtYd) (width 0.05))
+    (fp_line (start -1.41 1.54) (end -1.41 -1.54) (layer F.CrtYd) (width 0.05))
+    (fp_line (start 1.25 1.25) (end -1.25 1.25) (layer F.Fab) (width 0.1))
+    (fp_line (start 1.25 -1.25) (end 1.25 1.25) (layer F.Fab) (width 0.1))
+    (fp_line (start -0.5 -1.25) (end 1.25 -1.25) (layer F.Fab) (width 0.1))
+    (fp_line (start -1.25 1.25) (end -1.25 -0.5) (layer F.Fab) (width 0.1))
+    (fp_line (start -1.35 -1.2) (end -1.35 -1.45) (layer F.SilkS) (width 0.1))
+    (fp_line (start 1.35 -1.35) (end 1.35 -1.2) (layer F.SilkS) (width 0.1))
+    (fp_line (start 1.2 -1.35) (end 1.35 -1.35) (layer F.SilkS) (width 0.1))
+    (fp_line (start 1.35 1.35) (end 1.2 1.35) (layer F.SilkS) (width 0.1))
+    (fp_line (start 1.35 1.35) (end 1.35 1.2) (layer F.SilkS) (width 0.1))
+    (fp_line (start -1.35 1.35) (end -1.35 1.2) (layer F.SilkS) (width 0.1))
+    (fp_line (start -1.25 -0.5) (end -0.5 -1.25) (layer F.Fab) (width 0.1))
+    (fp_line (start -1.35 1.36) (end -1.2 1.36) (layer F.SilkS) (width 0.1))
+    (fp_text user %R (at 0 0 270) (layer F.Fab)
+      (effects (font (size 0.5 0.5) (thickness 0.075)))
+    )
+    (pad 5 smd rect (at 0.975 1.025) (size 0.5 0.35) (layers F.Cu F.Paste F.Mask))
+    (pad 6 smd rect (at 0.325 1.025) (size 0.5 0.35) (layers F.Cu F.Paste F.Mask))
+    (pad 7 smd rect (at -0.325 1.025) (size 0.5 0.35) (layers F.Cu F.Paste F.Mask))
+    (pad 8 smd rect (at -0.975 1.025) (size 0.5 0.35) (layers F.Cu F.Paste F.Mask))
+    (pad 1 smd rect (at -0.975 -1.025) (size 0.5 0.35) (layers F.Cu F.Paste F.Mask))
+    (pad 2 smd rect (at -0.325 -1.025) (size 0.5 0.35) (layers F.Cu F.Paste F.Mask))
+    (pad 3 smd rect (at 0.325 -1.025) (size 0.5 0.35) (layers F.Cu F.Paste F.Mask))
+    (pad 4 smd rect (at 0.975 -1.025) (size 0.5 0.35) (layers F.Cu F.Paste F.Mask))
+    (model ${KISYS3DMOD}/Package_LGA.3dshapes/Bosch_LGA-8_2.5x2.5mm_P0.65mm_ClockwisePinNumbering.wrl
+      (offset (xyz 0.01500000025472259 -0.03500000059435272 0))
+      (scale (xyz 1 1 1))
+      (rotate (xyz 0 0 0))
+    )
   )
   (gr_text GND (at 121.6 123.6) (layer F.SilkS)

Commit message: Going Open-Source
Need just a check before next prod
Parts:
- removed G1 (x2): LOGO, MWL:Serigraphie
- removed REF**: Bosch_LGA-8_2.5x2.5mm_P0.65mm_ClockwisePinNumbering, Package_LGA:Bosch_LGA-8_2.5x2.5mm_P0.65mm_ClockwisePinNumbering
- J1: value Conn_01x22_Male -> (none)
- J2: value Conn_01x18_Male -> (none)
- J3: value Conn_01x10_Male -> (none)
- J4, J5: value Prog -> (none)
- moved J4 7.78 mm to (127.5, 132.5)
Routing:
- net V_NRF: track 43.9 -> 52.5 mm
- net SWDIO: track 43.7 -> 51.8 mm
- net SWDCLK: track 47.3 -> 54.6 mm
- net GND: vias 29 -> 27
Other:
- board text added: "www.anderson69s.com"
