File: ADM_52840.sch (KiCad schematic (older format))
At the start: 8 parts, among them J1 Conn_01x22_Male, J2 Conn_01x18_Male, J3 Conn_01x10_Male, J4 Prog, J5 Prog, U1 HolyIOT_NRF52840

Commit message: Rename
Parts:
- removed G1: LOGO, MWL:Serigraphie, symbol Serigraphie:LOGO
- U1: footprint MWL:HolyIOT-NRF52840-Module -> LEGACY:HolyIOT-NRF52840-Module; symbol MWL:HolyIOT_NRF52840 -> Legacy:HolyIOT_NRF52840
Changed lines of the file:
@@
 EESchema Schematic File Version 4
-LIBS:HolyIoT-NRF52840-Breakout-cache
-EELAYER 26 0
+EELAYER 30 0
 EELAYER END
 $Descr A4 11693 8268
 encoding utf-8
 Sheet 1 1
-Title "Holy_IOT_NRF52840_BreakOut_Board"
-Date "2018-08-31"
+Title "ADM_52840"
+Date "2020-10-31"
 Rev "1.0"
-Comp "Mini World Lyon"
+Comp "Atelier Du Maker"
 Comment1 "Alexandre Perier-Muzet"
 Comment2 "Mickael Veleine"
-Comment3 "Aubrin Dodeller"
+Comment3 "Gaetan Noël"
 Comment4 ""
 $EndDescr
@@
 	4850 2050 4700 2050
 $Comp
-L MWL:HolyIOT_NRF52840 U1
+L Legacy:HolyIOT_NRF52840 U1
 U 1 1 5B9DD21A
 P 5750 3250
 F 0 "U1" H 5750 4265 50  0000 C CNN
 F 1 "HolyIOT_NRF52840" H 5750 4174 50  0000 C CNN
-F 2 "MWL:HolyIOT-NRF52840-Module" H 5750 3250 50  0001 C CNN
+F 2 "LEGACY:HolyIOT-NRF52840-Module" H 5750 3250 50  0001 C CNN
 F 3 "" H 5750 3250 50  0001 C CNN
 	1    5750 3250
@@
 Wire Wire Line
 	4850 4650 4850 4800
-$Comp
-L Serigraphie:LOGO G1
-U 1 1 5B9AE5DB
-P 5700 1500
-F 0 "G1" H 5700 1270 60  0001 C CNN
-F 1 "LOGO" H 5700 1730 60  0001 C CNN
-F 2 "MWL:Serigraphie" H 5700 1500 50  0001 C CNN
-F 3 "" H 5700 1500 50  0001 C CNN
-	1    5700 1500
-	1    0    0    -1
-$EndComp
 Wire Wire Line
 	5900 4000 5900 4200

Commit message: update
Parts:
- removed J1: Conn_01x22_Male, Connector_PinHeader_2.54mm:PinHeader_1x22_P2.54mm_Vertical, symbol Connector:Conn_01x22_Male
- removed J2: Conn_01x18_Male, Connector_PinHeader_2.54mm:PinHeader_1x18_P2.54mm_Vertical, symbol Connector:Conn_01x18_Male
- removed J3: Conn_01x10_Male, Connector_PinHeader_2.54mm:PinHeader_1x10_P2.54mm_Vertical, symbol Connector:Conn_01x10_Male
- removed J4: Prog, Connector_PinHeader_1.27mm:PinHeader_2x05_P1.27mm_Vertical_SMD, symbol Connector_Generic_MountingPin:Conn_02x05_Odd_Even_MountingPin
- added C1: 100nF, MWL:SM0805, symbol Device:C_Small
- added C3: 1nF, MWL:SM0805, symbol Device:C_Small
- added C4, C5, C6: 10microF, MWL:SM0805, symbol Device:C_Small
- added D1: LED1, symbol Device:LED
- added D2: LED2, symbol Device:LED
- added D3: LED3, symbol Device:LED
- added D4: MBR120, symbol Device:D_Schottky
- added D5: SK6812, symbol LEGACY:SK6812
- added J1: JST, symbol Connector:Conn_01x02_Male
- added J2: SK6812_OUT, LEGACY:PADS_CONNEXION, symbol Connector:Conn_01x01_Male
- added P1: USB_micro_B, symbol LEGACY:USB_micro_B
- added Q1: DMP2045U//DMG3415U-7, Package_SON:Diodes_PowerDI3333-8, symbol Transistor_FET:DMP3013SFV
- added R1: 806K, symbol Device:R
- added R2: 2M, symbol Device:R
- added R3: 10K, symbol Device:R
- added R4: 1K, symbol Device:R
- added R5, R6: 100K, symbol Device:R
- added SW1: BTN1, symbol Switch:SW_Push
- added SW2: BTN2, symbol Switch:SW_Push
- added SW3: RESET, symbol Switch:SW_Push
- added U2: MX25R3235FZNxx1, Package_SON:WSON-8-1EP_6x5mm_P1.27mm_EP3.4x4mm, symbol Memory_Flash:MX25R3235FZNxx1
- added U3: MCP73831, symbol LEGACY:MCP73831
- added U4: AP2127K-3.3, Package_TO_SOT_SMD:SOT-23-5, symbol Regulator_Linear:AP2127K-3.3
- C2: value C -> 10microF
- U1: symbol Legacy:HolyIOT_NRF52840 -> LEGACY:HolyIOT_NRF52840
Connections:
- net labels added: D+, D-, QSPI_0, QSPI_1, QSPI_2, QSPI_3, QSPI_CLK, QSPI_CS, SK_SIGNAL, VBAT, VBUS
- wire segments 212 -> 267
- no-connect marks 7 -> 1
Other:
- note added: "BAT JST"
- note added: "Charge Lipo"
- note added: "Flash SPI"
- note added: "LDO"
- note added: "Micro-USB"
- note added: "Program 2.54mm"
- note added: "SK6812"
- note removed: "Program 2.54mm Format"
- note removed: "Program CMS Format"
- moved on the sheet: C2, J5

Commit message: update spi
Parts:
- C1, C3: footprint MWL:SM0805 -> LEGACY:SM0603
- C2, C4, C5, C6: footprint MWL:SM0805 -> LEGACY:SM0805
- D1, D2, D3, R1, R2, R3, R4, R5, R6: footprint (none) -> LEGACY:SM0805
- D5: footprint (none) -> LEGACY:WS2812B; symbol LEGACY:SK6812 -> ADM_52840-rescue:SK6812-LEGACY
- J1: footprint (none) -> Connectors_JST:JST_PH_S2B-PH-SM4-TB_02x2.00mm_Angled
- P1: footprint (none) -> LEGACY:USB_Micro-B; symbol LEGACY:USB_micro_B -> ADM_52840-rescue:USB_micro_B-LEGACY
- SW1, SW2, SW3: footprint (none) -> LEGACY:SWITCH_CMS
- U1: symbol LEGACY:HolyIOT_NRF52840 -> ADM_52840-rescue:HolyIOT_NRF52840-LEGACY
- U2: value MX25R3235FZNxx1 -> MX25R6435F
- U3: footprint (none) -> LEGACY:SOT23-5; symbol LEGACY:MCP73831 -> ADM_52840-rescue:MCP73831-LEGACY
- U4: footprint Package_TO_SOT_SMD:SOT-23-5 -> LEGACY:SOT23-5; symbol Regulator_Linear:AP2127K-3.3 -> ADM_52840-rescue:AP2127K-3.3-Regulator_Linear
Changed lines of the file:
@@
 	3775 2000 3625 2000
 $Comp
-L LEGACY:HolyIOT_NRF52840 U1
+L ADM_52840-rescue:HolyIOT_NRF52840-LEGACY U1
 U 1 1 5B9DD21A
 P 4675 3200
@@
 	5525 4100 6575 4100
 Wire Wire Line
-	5775 3675 6575 3675
+	5775 3675 5950 3675
 Wire Wire Line
 	5850 3550 6575 3550
@@
 F 0 "C2" H 3550 4475 50  0000 L CNN
 F 1 "10microF" H 3400 4575 50  0000 L CNN
-F 2 "MWL:SM0805" H 3813 4350 50  0001 C CNN
+F 2 "LEGACY:SM0805" H 3813 4350 50  0001 C CNN
 F 3 "~" H 3775 4500 50  0001 C CNN
 	1    3775 4500
@@
 F 0 "SW3" H 4750 5100 50  0000 L CNN
 F 1 "RESET" H 4850 5250 50  0000 L CNN
-F 2 "" H 4825 5350 50  0001 C CNN
+F 2 "LEGACY:SWITCH_CMS" H 4825 5350 50  0001 C CNN
 F 3 "~" H 4825 5350 50  0001 C CNN
 	1    4825 5150
@@
 F 0 "SW1" H 2875 2250 50  0000 C CNN
 F 1 "BTN1" H 2750 2400 50  0000 C CNN
-F 2 "" H 2875 2500 50  0001 C CNN
+F 2 "LEGACY:SWITCH_CMS" H 2875 2500 50  0001 C CNN
 F 3 "~" H 2875 2500 50  0001 C CNN
 	1    2875 2300
@@
 $EndComp
 $Comp
-L LEGACY:USB_micro_B P1
+L ADM_52840-rescue:USB_micro_B-LEGACY P1
 U 1 1 5F9E1D2D
 P 5050 7325
 F 0 "P1" V 5075 7275 60  0000 L CNN
 F 1 "USB_micro_B" V 5225 7025 60  0000 L CNN
-F 2 "" H 5050 7325 60  0000 C CNN
+F 2 "LEGACY:USB_Micro-B" H 5050 7325 60  0001 C CNN
 F 3 "" H 5050 7325 60  0000 C CNN
 	1    5050 7325
@@
 F 0 "D1" H 2650 3250 50  0000 C CNN
 F 1 "LED1" H 2425 3150 50  0000 C CNN
-F 2 "" H 2525 3300 50  0001 C CNN
+F 2 "LEGACY:SM0805" H 2525 3300 50  0001 C CNN
 F 3 "~" H 2525 3300 50  0001 C CNN
 	1    2525 3300
@@
 F 0 "SW2" H 2325 2350 50  0000 C CNN
 F 1 "BTN2" H 2200 2500 50  0000 C CNN
-F 2 "" H 2325 2600 50  0001 C CNN
+F 2 "LEGACY:SWITCH_CMS" H 2325 2600 50  0001 C CNN
 F 3 "~" H 2325 2600 50  0001 C CNN
 	1    2325 2400
@@
 P 9750 1475
 F 0 "U2" H 9150 1925 50  0000 L CNN
-F 1 "MX25R3235FZNxx1" H 9100 1850 50  0000 L CNN
+F 1 "MX25R6435F" H 9100 1850 50  0000 L CNN
 F 2 "Package_SON:WSON-8-1EP_6x5mm_P1.27mm_EP3.4x4mm" H 9750 875 50  0001 C CNN
 F 3 "http://www.macronix.com/Lists/Datasheet/Attachments/7534/MX25R3235F,%20Wide%20Range,%2032Mb,%20v1.6.pdf" H 9750 1475 50  0001 C CNN
@@
 F 0 "C1" H 10400 1050 50  0000 L CNN
 F 1 "100nF" H 10400 975 50  0000 L CNN
-F 2 "MWL:SM0805" H 10338 850 50  0001 C CNN
+F 2 "LEGACY:SM0603" H 10338 850 50  0001 C CNN
 F 3 "~" H 10300 1000 50  0001 C CNN
 	1    10300 1000
@@
 F 0 "D2" H 3000 3350 50  0000 C CNN
 F 1 "LED2" H 2825 3250 50  0000 C CNN
-F 2 "" H 2875 3400 50  0001 C CNN
+F 2 "LEGACY:SM0805" H 2875 3400 50  0001 C CNN
 F 3 "~" H 2875 3400 50  0001 C CNN
 	1    2875 3400
@@
 Text GLabel 9150 1475 0    50   Input ~ 0
 QSPI_CS
-Text GLabel 5775 3825 2    50   Input ~ 0
+Text GLabel 5950 3675 2    50   Input ~ 0
 QSPI_0
 Wire Wire Line
 	5475 3500 5725 3500
 Text GLabel 6250 3075 2    50   Input ~ 0
-QSPI_1
+QSPI_2
+Wire Wire Line
+	4625 3950 4625 4250
+Wire Wire Line
+	4625 4250 4525 4250
+Wire Wire Line
+	4525 4250 4525 4525
 Text GLabel 4525 4525 3    50   Input ~ 0
-QSPI_2
-Wire Wire Line
-	4625 3950 4625 4250
-Wire Wire Line
-	4625 4250 4525 4250
-Wire Wire Line
-	4525 4250 4525 4525
-Text GLabel 4650 4525 3    50   Input ~ 0
 QSPI_3
 Wire Wire Line
@@
 	4750 4400 4750 4525
 $Comp
-L LEGACY:MCP73831 U3
+L ADM_52840-rescue:MCP73831-LEGACY U3
 U 1 1 601FBD0A
 P 9700 3475
 F 0 "U3" H 9725 3962 60  0000 C CNN
 F 1 "MCP73831" H 9725 3856 60  0000 C CNN
-F 2 "" H 9700 3475 60  0000 C CNN
+F 2 "LEGACY:SOT23-5" H 9700 3475 60  0001 C CNN
 F 3 "" H 9700 3475 60  0000 C CNN
 	1    9700 3475
@@
 F 0 "J1" H 6525 6950 50  0000 C CNN
 F 1 "JST" H 6525 7275 50  0000 C CNN
-F 2 "" H 6525 7175 50  0001 C CNN
+F 2 "Connectors_JST:JST_PH_S2B-PH-SM4-TB_02x2.00mm_Angled" H 6525 7175 50  0001 C CNN
 F 3 "~" H 6525 7175 50  0001 C CNN
 	1    6525 7175
@@
 F 0 "R4" V 9000 3675 50  0000 C CNN
 F 1 "1K" V 9100 3675 50  0000 C CNN
-F 2 "" V 9030 3675 50  0001 C CNN
+F 2 "LEGACY:SM0805" V 9030 3675 50  0001 C CNN
 F 3 "~" H 9100 3675 50  0001 C CNN
 	1    9100 3675
@@
 F 0 "D3" H 8850 3625 50  0000 C CNN
 F 1 "LED3" H 8625 3525 50  0000 C CNN
-F 2 "" H 8725 3675 50  0001 C CNN
+F 2 "LEGACY:SM0805" H 8725 3675 50  0001 C CNN
 F 3 "~" H 8725 3675 50  0001 C CNN
 	1    8725 3675
@@
 F 0 "R3" V 10200 3475 50  0000 C CNN
 F 1 "10K" V 10300 3475 50  0000 C CNN
-F 2 "" V 10230 3475 50  0001 C CNN
+F 2 "LEGACY:SM0805" V 10230 3475 50  0001 C CNN
 F 3 "~" H 10300 3475 50  0001 C CNN
 	1    10300 3475
@@
 F 0 "C4" H 10700 3425 50  0000 L CNN
 F 1 "10microF" V 10750 3000 50  0000 L CNN
-F 2 "MWL:SM0805" H 10638 3225 50  0001 C CNN
+F 2 "LEGACY:SM0805" H 10638 3225 50  0001 C CNN
 F 3 "~" H 10600 3375 50  0001 C CNN
 	1    10600 3375
@@
 F 0 "R2" V 1450 3200 50  0000 C CNN
 F 1 "2M" V 1550 3200 50  0000 C CNN
-F 2 "" V 1480 3200 50  0001 C CNN
+F 2 "LEGACY:SM0805" V 1480 3200 50  0001 C CNN
 F 3 "~" H 1550 3200 50  0001 C CNN
 	1    1550 3200
@@
 F 0 "C3" H 1925 3225 50  0000 L CNN
 F 1 "1nF" H 1925 3125 50  0000 L CNN
-F 2 "MWL:SM0805" H 1863 3025 50  0001 C CNN
+F 2 "LEGACY:SM0603" H 1863 3025 50  0001 C CNN
 F 3 "~" H 1825 3175 50  0001 C CNN
 	1    1825 3175
@@
 F 0 "R1" V 1450 2800 50  0000 C CNN
 F 1 "806K" V 1550 2800 50  0000 C CNN
-F 2 "" V 1480 2800 50  0001 C CNN
+F 2 "LEGACY:SM0805" V 1480 2800 50  0001 C CNN
 F 3 "~" H 1550 2800 50  0001 C CNN
 	1    1550 2800
@@
 	5725 3500 5725 3825
 $Comp
-L Regulator_Linear:AP2127K-3.3 U4
+L ADM_52840-rescue:AP2127K-3.3-Regulator_Linear U4
 U 1 1 60B8E04E
 P 10300 5450
 F 0 "U4" H 10300 5792 50  0000 C CNN
 F 1 "AP2127K-3.3" H 10300 5701 50  0000 C CNN
-F 2 "Package_TO_SOT_SMD:SOT-23-5" H 10300 5775 50  0001 C CNN
+F 2 "LEGACY:SOT23-5" H 10300 5775 50  0001 C CNN
 F 3 "https://www.diodes.com/assets/Datasheets/AP2127.pdf" H 10300 5550 50  0001 C CNN
 	1    10300 5450
@@
 F 0 "C5" H 9150 5450 50  0000 L CNN
 F 1 "10microF" H 8975 5350 50  0000 L CNN
-F 2 "MWL:SM0805" H 9388 5300 50  0001 C CNN
+F 2 "LEGACY:SM0805" H 9388 5300 50  0001 C CNN
 F 3 "~" H 9350 5450 50  0001 C CNN
 	1    9350 5450
@@
 F 0 "C6" H 10550 5450 50  0000 L CNN
 F 1 "10microF" V 10800 5425 50  0000 L CNN
-F 2 "MWL:SM0805" H 10713 5375 50  0001 C CNN
+F 2 "LEGACY:SM0805" H 10713 5375 50  0001 C CNN
 F 3 "~" H 10675 5525 50  0001 C CNN
 	1    10675 5525
@@
 F 0 "R6" V 8325 5575 50  0000 C CNN
 F 1 "100K" V 8425 5575 50  0000 C CNN
-F 2 "" V 8355 5575 50  0001 C CNN
+F 2 "LEGACY:SM0805" V 8355 5575 50  0001 C CNN
 F 3 "~" H 8425 5575 50  0001 C CNN
 	1    8425 5575
@@
 F 0 "R5" V 9875 5450 50  0000 C CNN
 F 1 "100K" V 9775 5450 50  0000 C CNN
-F 2 "" V 9705 5450 50  0001 C CNN
+F 2 "LEGACY:SM0805" V 9705 5450 50  0001 C CNN
 F 3 "~" H 9775 5450 50  0001 C CNN
 	1    9775 5450
@@
 	2425 6550 2425 7750
 $Comp
-L LEGACY:SK6812 D5
+L ADM_52840-rescue:SK6812-LEGACY D5
 U 1 1 6166925D
 P 1375 6875
 F 0 "D5" H 1400 7050 60  0000 C CNN
 F 1 "SK6812" H 1400 6650 60  0000 C CNN
-F 2 "" H 1375 6875 60  0000 C CNN
+F 2 "LEGACY:WS2812B" H 1375 6875 60  0001 C CNN
 F 3 "" H 1375 6875 60  0000 C CNN
 	1    1375 6875
@@
 Wire Wire Line
 	825  6975 825  7175
+Text GLabel 5775 3825 2    50   Input ~ 0
+QSPI_CS
+Text GLabel 4650 4525 3    50   Input ~ 0
+QSPI_1
 $EndSCHEMATC

Commit message: update
Parts:
- U1: symbol ADM_52840-rescue:HolyIOT_NRF52840-LEGACY -> LEGACY:HolyIOT_NRF52840
- U2: value MX25R6435F -> GD25Q16
Connections:
- net labels added: P0.31
- wire segments 267 -> 160
Other:
- note added: "MONITOR BAT"
- moved on the sheet: C2, C3, D1, D2, D3, R1, R2, SW1, SW2, SW3, U1

Commit message: SAV
Parts:
- added J3: Conn_01x14_Male, Connector_PinSocket_2.54mm:PinSocket_1x14_P2.54mm_Horizontal, symbol Connector:Conn_01x14_Male
- added J4: Conn_01x16_Male, Connector_PinSocket_2.54mm:PinSocket_1x16_P2.54mm_Vertical, symbol Connector:Conn_01x16_Male
- added J6: Conn_01x03_Male, Connector_PinSocket_2.54mm:PinSocket_1x03_P2.54mm_Vertical, symbol Connector:Conn_01x03_Male
- D4: footprint (none) -> LEGACY:SOD-123
- J2: footprint LEGACY:PADS_CONNEXION -> LEGACY:pin_array_3x1; symbol Connector:Conn_01x01_Male -> Connector:Conn_01x03_Male
- J5: footprint Connector_PinHeader_2.54mm:PinHeader_1x06_P2.54mm_Vertical -> Connector_PinSocket_2.54mm:PinSocket_2x03_P2.54mm_Vertical
- Q1: value DMP2045U//DMG3415U-7 -> DMP2045U; footprint Package_SON:Diodes_PowerDI3333-8 -> LEGACY:SOT23
- U2: footprint Package_SON:WSON-8-1EP_6x5mm_P1.27mm_EP3.4x4mm -> LEGACY:SON80P400X300X60-10N
Connections:
- wire segments 160 -> 245
Other:
- moved on the sheet: C2, D1, D2, SW1, SW2, SW3, U1

Commit message: route & 3D
Parts:
- removed J6: Conn_01x03_Male, Connector_PinSocket_2.54mm:PinSocket_1x03_P2.54mm_Vertical, symbol Connector:Conn_01x03_Male
- added R7, R8: 330, LEGACY:SM0603, symbol Device:R
- D1, D2, D3, R1, R2, R3, R4, R5, R6: footprint LEGACY:SM0805 -> LEGACY:SM0603
- J1: footprint Connectors_JST:JST_PH_S2B-PH-SM4-TB_02x2.00mm_Angled -> Connector_JST:JST_PH_S2B-PH-SM4-TB_1x02-1MP_P2.00mm_Horizontal
- J3: value Conn_01x14_Male -> Conn_01x15_Male; footprint Connector_PinSocket_2.54mm:PinSocket_1x14_P2.54mm_Horizontal -> Connector_PinSocket_2.54mm:PinSocket_1x15_P2.54mm_Vertical; symbol Connector:Conn_01x14_Male -> Connector:Conn_01x15_Male
- J4: value Conn_01x16_Male -> Conn_01x19_Male; footprint Connector_PinSocket_2.54mm:PinSocket_1x16_P2.54mm_Vertical -> Connector_PinSocket_2.54mm:PinSocket_1x18_P2.54mm_Vertical; symbol Connector:Conn_01x16_Male -> Connector:Conn_01x18_Male
- J5: value Prog -> JTAG
- U3: footprint LEGACY:SOT23-5 -> Package_TO_SOT_SMD:SOT-23-5
Connections:
- wire segments 245 -> 258
Other:
- moved on the sheet: D1, D2, SW1, SW2

Commit message: 3D
Parts:
- U1: symbol LEGACY:HolyIOT_NRF52840 -> ADM_52840-rescue:HolyIOT_NRF52840-LEGACY
- U3: footprint Package_TO_SOT_SMD:SOT-23-5 -> LEGACY:SOT23-5
Changed lines of the file:
@@
 $EndDescr
 $Comp
-L LEGACY:HolyIOT_NRF52840 U1
+L ADM_52840-rescue:HolyIOT_NRF52840-LEGACY U1
 U 1 1 5B9DD21A
 P 4625 2275
@@
 F 0 "U3" H 9725 3962 60  0000 C CNN
 F 1 "MCP73831" H 9725 3856 60  0000 C CNN
-F 2 "Package_TO_SOT_SMD:SOT-23-5" H 9700 3475 60  0001 C CNN
+F 2 "LEGACY:SOT23-5" H 9700 3475 60  0001 C CNN
 F 3 "" H 9700 3475 60  0000 C CNN
 	1    9700 3475

Commit message: update alim
Parts:
- Q1: symbol Transistor_FET:DMP3013SFV -> Transistor_FET:AO3401A
Connections:
- net VBAT: now also Q1.3 (D); no longer Q1.5 (D)
- net VBUS: now also Q1.1 (G); no longer Q1.4 (G)
- net at D2.1 (K): now also R8.1
- net at C5.1, D4.1 (K), Q1.2 (S)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: no longer Q1.1 (S), Q1.3 (S)
Changed lines of the file:
@@
 $EndComp
 $Comp
-L Transistor_FET:DMP3013SFV Q1
+L Transistor_FET:AO3401A Q1
 U 1 1 60C00813
 P 8875 5000
@@
 Wire Wire Line
 	1900 2075 3525 2075
+Wire Wire Line
+	1600 2075 1500 2075
 $EndSCHEMATC
